File: eagle/Temperature-Humidity/Temperature-Humidity.brd (EAGLE design)
At the start: 25 x 25 mm, 5 parts, among them U1 SHT1x

Commit message: Proto boards library 0.1
Parts:
- removed U$1: (no value), theairboard:BRD_FRAME
- added FRAME1: SCH_FRAME, theairboard:BOARD_FRAME
Changed lines of the file:
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@@
 <attribute name="VALUE" x="9.918" y="15.694" size="1.27" layer="25" rot="R90"/>
 </element>
-<element name="U$1" library="theairboard" package="BRD_FRAME" value="" x="-59.69" y="-53.34"/>
 <element name="U$2" library="theairboard" package="LAYOUT25X25" value="" x="0" y="0"/>
+<element name="FRAME1" library="theairboard" package="BOARD_FRAME" value="SCH_FRAME" x="-104" y="-73"/>
 </elements>
 <signals>
