File: breakout boards/MotorBoard/MotorBoard.brd (EAGLE design)
At the start: 25 x 25 mm, 10 parts, among them Q1 FDG6303N

Commit message: updated breakout boards
Parts:
- D1, D2: device theairboard:DO-214AC -> TheAirBoard_breakouts:DO-214AC
- JP1: device theairboard:SIL-1X10 -> TheAirBoard_breakouts:SIL10-2.54MM
- Q1: device theairboard:SC70-6 -> TheAirBoard_breakouts:SC70-6
Changed lines of the file:
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@@
 </plain>
 <attributes>
-<attribute name="DESIGNER" value="theairboard.cc"/>
+<attribute name="DESIGNER" value="AirThings Inc"/>
 <attribute name="REV" value="1.0"/>
 <attribute name="SENSOR" value="Dual motor drive"/>
@@
 </autorouter>
 <elements>
-<element name="JP1" library="theairboard" package="SIL-1X10" value="SIL" x="38.1" y="20.32" smashed="yes" rot="R180">
-<attribute name="OC_NEWARK" value="93K5133" x="11.43" y="57.15" size="1.778" layer="27" rot="R180" display="off"/>
+<element name="JP1" library="TheAirBoard_breakouts" package="SIL10-2.54MM" value="SIL" x="38.1" y="20.32" smashed="yes" rot="R180">
 <attribute name="MANUFACTURER" value="FCI" x="11.43" y="57.15" size="1.778" layer="27" rot="R180" display="off"/>
-<attribute name="OC_FARNELL" value="1097958" x="11.43" y="57.15" size="1.778" layer="27" rot="R180" display="off"/>
 <attribute name="PART_NUMBER" value="77315-818-36LF " x="11.43" y="57.15" size="1.778" layer="27" rot="R180" display="off"/>
+<attribute name="FARNELL" value="1097958" x="38.1" y="20.32" size="1.778" layer="27" rot="R180" display="off"/>
+<attribute name="DESCRIPTION" value="Thru-hole, right angle, male, 1 row, 10-way, 2.54mm" x="38.1" y="20.32" size="1.778" layer="27" rot="R180" display="off"/>
+<attribute name="DATASHEET" value="www.farnell.com/datasheets/8281.pdf" x="38.1" y="20.32" size="1.778" layer="27" rot="R180" display="off"/>
+<attribute name="NEWARK" value="93K5133" x="38.1" y="20.32" size="1.778" layer="27" rot="R180" display="off"/>
 </element>
 <element name="FRAME1" library="theairboard" package="BOARD_FRAME" value="SCH_FRAME" x="-45.72" y="-55.88"/>
-<element name="Q1" library="theairboard" package="SC70-6" value="FDG6303N" x="43.18" y="24.13" smashed="yes" rot="R90">
-<attribute name="DESCRIPTION" value="Dual N-Channel, Digital FET" x="78.74" y="67.31" size="1.778" layer="27" rot="R90" display="off"/>
+<element name="Q1" library="TheAirBoard_breakouts" package="SC70-6" value="FDG6303N" x="43.18" y="24.13" smashed="yes" rot="R90">
+<attribute name="DESCRIPTION" value="" x="78.74" y="67.31" size="1.778" layer="27" rot="R90" display="off"/>
 <attribute name="MANUFACTURER" value="FAIRCHILD" x="78.74" y="67.31" size="1.778" layer="27" rot="R90" display="off"/>
 <attribute name="PART_NUMBER" value="FDG6303N" x="78.74" y="67.31" size="1.778" layer="27" rot="R90" display="off"/>
 <attribute name="VALUE" x="41.432" y="23.634" size="1.016" layer="25" rot="R180"/>
+<attribute name="FARNELL" value="1611233" x="43.18" y="24.13" size="1.778" layer="27" rot="R90" display="off"/>
+<attribute name="DATASHEET" value="www.farnell.com/datasheets/169519.pdf" x="43.18" y="24.13" size="1.778" layer="27" rot="R90" display="off"/>
+<attribute name="NEWARK" value="58K1450" x="43.18" y="24.13" size="1.778" layer="27" rot="R90" display="off"/>
 </element>
 <element name="U$1" library="theairboard" package="LAYOUT25X25" value="" x="25.4" y="10.16"/>
@@
 <element name="JP4" library="SparkFun-Connectors" package="1X01NS" value="M01SMDNS" x="34.925" y="30.75"/>
 <element name="JP5" library="SparkFun-Connectors" package="1X01NS" value="M01SMDNS" x="41.245" y="30.74"/>
-<element name="D1" library="theairboard" package="DO-214AC" value="S1M" x="43.942" y="27.94" smashed="yes" rot="R180">
-<attribute name="OC_NEWARK" value="58K2390" x="43.942" y="27.94" size="1.778" layer="27" rot="R180" display="off"/>
-<attribute name="MANUFACTURER" value="Fairchild" x="43.942" y="27.94" size="1.778" layer="27" rot="R180" display="off"/>
-<attribute name="OC_FARNELL" value="9843841" x="43.942" y="27.94" size="1.778" layer="27" rot="R180" display="off"/>
+<element name="D1" library="TheAirBoard_breakouts" package="DO-214AC" value="S1M" x="43.942" y="27.94" smashed="yes" rot="R180">
+<attribute name="MANUFACTURER" value="FAIRCHILD" x="43.942" y="27.94" size="1.778" layer="27" rot="R180" display="off"/>
 <attribute name="PART_NUMBER" value="S1M" x="43.942" y="27.94" size="1.778" layer="27" rot="R180" display="off"/>
-</element>
-<element name="D2" library="theairboard" package="DO-214AC" value="S1M" x="36.068" y="27.94" smashed="yes" rot="R180">
-<attribute name="OC_NEWARK" value="58K2390" x="36.068" y="27.94" size="1.778" layer="27" rot="R180" display="off"/>
-<attribute name="MANUFACTURER" value="Fairchild" x="36.068" y="27.94" size="1.778" layer="27" rot="R180" display="off"/>
-<attribute name="OC_FARNELL" value="9843841" x="36.068" y="27.94" size="1.778" layer="27" rot="R180" display="off"/>
+<attribute name="FARNELL" value="9843841" x="43.942" y="27.94" size="1.778" layer="27" rot="R180" display="off"/>
+<attribute name="DESCRIPTION" value="1A, equivalent to 1N4007" x="43.942" y="27.94" size="1.778" layer="27" rot="R180" display="off"/>
+<attribute name="DATASHEET" value="www.farnell.com/datasheets/1766308.pdf" x="43.942" y="27.94" size="1.778" layer="27" rot="R180" display="off"/>
+<attribute name="NEWARK" value="58K2390" x="43.942" y="27.94" size="1.778" layer="27" rot="R180" display="off"/>
+</element>
+<element name="D2" library="TheAirBoard_breakouts" package="DO-214AC" value="S1M" x="36.068" y="27.94" smashed="yes" rot="R180">
+<attribute name="MANUFACTURER" value="FAIRCHILD" x="36.068" y="27.94" size="1.778" layer="27" rot="R180" display="off"/>
 <attribute name="PART_NUMBER" value="S1M" x="36.068" y="27.94" size="1.778" layer="27" rot="R180" display="off"/>
+<attribute name="FARNELL" value="9843841" x="36.068" y="27.94" size="1.778" layer="27" rot="R180" display="off"/>
+<attribute name="DESCRIPTION" value="1A, equivalent to 1N4007" x="36.068" y="27.94" size="1.778" layer="27" rot="R180" display="off"/>
+<attribute name="DATASHEET" value="www.farnell.com/datasheets/1766308.pdf" x="36.068" y="27.94" size="1.778" layer="27" rot="R180" display="off"/>
+<attribute name="NEWARK" value="58K2390" x="36.068" y="27.94" size="1.778" layer="27" rot="R180" display="off"/>
 </element>
 </elements>
